File: power.kicad_sch (KiCad schematic)
At the start: 33 parts, among them J1 Conn_01x02_Pin, J2 USB_C_Receptacle_PowerOnly_6P, J3 Conn_01x03_Pin, Q6 DTC143Z, U1 BQ24073RGTR, U2 TPD1E10B06DPYR, U3 TPD1E10B06DPYR, U4 TPD1E10B06DPYR, U5 TPS61022RWUR, U7 AP2112K-1.8

Commit message: v4.4
Parts:
- C1, C8: value 4.7uF -> 4.7u
- C17, C5, C6: value 1uF -> 1u
- C18: value 10pF -> 100n; footprint Capacitor_SMD:C_0402_1005Metric -> Capacitor_SMD:C_0603_1608Metric; coef C0G -> (none)
- C2: value 10uF -> 22u
- C3, C4: value 22uF -> 22u
- C7: value 0.1uF -> 100n
- L1: value 1.0uh -> 1.5uh; footprint Inductor_SMD:L_1008_2520Metric -> Inductor_SMD:L_Changjiang_FTC322512S
- R6: value 750k -> 1M
- U5: footprint Muffin_SMD:RWU0007A -> Muffin_SMD:DSJ14_2P85X1P58; symbol Muffin_DC-DC:TPS61022RWUR -> Muffin_DC-DC:TPS63020DSJR; LCSC C915088 -> C15483
Connections:
- net +5V5: now also U5.4 (VOUT), U5.5 (VOUT); no longer C18.1, U5.3 (VOUT)
- net BOOST_FB: now also U5.3 (FB); no longer C18.2, U5.4 (FB)
- net EN_SERVO: now also U5.12 (EN); no longer U5.5 (EN)
- net GND: now also C18.2, U5.13 (PS/SYNC), U5.15 (EPAD), U5.2 (GND); no longer U5.1 (GND), U5.6 (MODE)
- net VSYS: now also U5.10 (VIN), U5.11 (VIN); no longer L1.1, U5.7 (VIN)
- net BOOST_SW renamed LY
- net LY: now also U5.6 (L2), U5.7 (L2); no longer U5.2 (SW)
- new net: C18.1, U5.1 (VINA)
- new net LX: L1.1, U5.8 (L1), U5.9 (L1)
- no-connect marks 0 -> 1
Other:
- note added: "Vout config R1 = R2 * (Vout/Vref - 1) Vref = 0.5v R2 < 200k Vout R1 R2 5V5 1M 100k"
- note removed: "Inductor: Vin 3.00...4.40 L = 1 uH Fsw 1.10...0.90 --------------------------------------- D = 1 - (Vin * n)/Vout = 0.47...0.22 Idc = (Vout * Iout)/(Vin * n) = 2.83...1.93 Ipp = (Vin * D)/(L*Fsw) = 1.55...0.87 Ip = Idc + Ipp/2 = 3.60...2.37 Chosen inductor: FWP252012P-1R0ML"
- note removed: "Operating conditions: Iout < 1.5A Vout = 5.1V Vin > 3.0V < 4.4V Fsw > 0.9MHz < 1.1Mhz n ~ 0.9"
- note removed: "Vout config R1 = R2 * (Vout/Vref - 1) Vref = 0.6v R2 < 300k Vout R1 R2 5V1 750k 100k"
- moved on the sheet: C18, C2, C3, C4, L1, R2, R6, U2, U3
